File: thundipiswitch2/tp_radio_board v4/tp_radio_board.kicad_pcb (KiCad board)
At the start: 2 copper layers, 99.9 x 94.6 mm, 87 parts, among them J1 FTSH-105-01-L-DV-K, J10 Conn_01x01_Male, J11 Conn_01x05_Male, J2 Conn_01x01_Male, J3 Conn_01x01_Male, J4 Conn_01x01_Male, J5 Conn_01x01_Male, J6 Conn_01x01_Male, J7 Conn_01x01_Male, J8 Conn_01x01_Male, J9 RJ12, K1 G5RL-K1-E_DC5, K2 G5RL-K1-E_DC5, K3 G5RL-K1-E_DC5, Q1 MMBT5551L, Q10 MMBT5551L, Q11 MMBT5551L, Q12 MMBT5551L, Q2 MMBT5551L, Q3 MMBT5551L, Q4 MMBT5551L, Q5 MMBT5551L, Q6 MMBT5551L, Q7 MMBT5551L, Q8 MMBT5551L, Q9 MMBT5551L, U1 BGM220PC22WGA2, U2 INA3221, U3 OKI-78SR-5_1.5-W36-C, U4 LP3982ILD-ADJ, U5 SI527DJ, U6 SI527DJ

Commit message: updates to board 3.1
Parts:
- moved C6 1.27 mm to (31.6, 119.0)
- moved R27 0.49 mm to (34.9, 117.0)
- moved R29 0.35 mm to (33.4, 116.8)
Routing:
- net GND: track 193.1 -> 238.2 mm, vias 220 -> 226
- net +5V: track 174.9 -> 202.9 mm, vias 15 -> 17
- net Net-(R29-Pad2): track 5.66 -> 8.35 mm, vias 0 -> 2
- net Net-(R5-Pad2): track 74.2 -> 76.4 mm
- net Net-(BT1-Pad1): track 55.2 -> 53.3 mm
- net +3V3: track 243.9 -> 245.6 mm
- net /Relay3_SET: track 64.2 -> 65.7 mm
- net /Relay2_UNSET: track 88.7 -> 90.0 mm
- net Net-(R27-Pad2): track 5.43 -> 6.61 mm
- net /INDICATOR2: track 23.9 -> 24.7 mm
- net /Relay3_UNSET: track 63.3 -> 64.0 mm
- net Net-(R5-Pad3): track 77.4 -> 78.0 mm
- net /INDICATOR3: track 10.9 -> 11.4 mm
- net /INDICATOR1: track 22.2 -> 22.7 mm, vias 5 -> 4
Other:
- outline, holes or cut-outs redrawn
- net class Default: clearance 0.1 -> 0.2
- rule trace_clearance: 0.1 -> 0.2
